File: backplane.brd (EAGLE design)
At the start: 170 x 80 mm, 8 parts, among them J1 5535070-4, J2 5535070-4, J3 5535070-4, J4 5535070-4, J5 5535070-4, J6 5535070-4, J7 5535070-4, J8 5535070-4

Commit message: routed the wires between backplane connectors, and alligned them with the centers
Parts:
- moved J1 7.08 mm to (18.0, 59.0)
- moved J2 7.08 mm to (38.3, 59.0)
- moved J3 7.08 mm to (58.6, 59.0)
- moved J4 7.08 mm to (79.0, 59.0)
- moved J5 7.08 mm to (99.3, 59.0)
- moved J6 7.08 mm to (119.6, 59.0)
- moved J7 7.08 mm to (139.9, 59.0)
- moved J8 7.08 mm to (160.2, 59.0)
Connections:
- net N$10 renamed SS_3
- net N$11 renamed SS_5
- net N$12 renamed SS_4
- net N$13 renamed SS_6
- net N$14 renamed SS_7
- net N$15 renamed EXT_1
- net N$17 renamed EXT_2
- net N$24 renamed SS_8
- net N$25 renamed SS_9
- net N$26 renamed SS_10
- net N$27 renamed SS_11
- net N$28 renamed SS_12
- net N$29 renamed SS_13
- net N$30 renamed SS_14
- net N$31 renamed EXT_3
- net N$32 renamed EXT_4
- net N$38 renamed 3.3V
- net N$40 renamed SCK
- net N$41 renamed MISO
- net N$42 renamed MOSI
- net N$43 renamed SDA
- net N$44 renamed SCL
- net N$45 renamed SS_15
- net N$46 renamed EXT_5
- net N$47 renamed EXT_6
- net N$48 renamed EXT_7
- net N$8 renamed SS_1
- net N$9 renamed SS_2
- removed net N$1: J1.A1, J2.A1, J3.A1, J4.A1, J5.A1, J6.A1, J7.A1, J8.A1
- removed net N$16: J1.B1, J2.B1, J3.B1, J4.B1, J5.B1, J6.B1, J7.B1, J8.B1
- removed net N$18: J1.B2, J2.B2, J3.B2, J4.B2, J5.B2, J6.B2, J7.B2, J8.B2
- removed net N$19: J1.B3, J2.B3, J3.B3, J4.B3, J5.B3, J6.B3, J7.B3, J8.B3
- removed net N$2: J1.A2, J2.A2, J3.A2, J4.A2, J5.A2, J6.A2, J7.A2, J8.A2
- removed net N$20: J1.B4, J2.B4, J3.B4, J4.B4, J5.B4, J6.B4, J7.B4, J8.B4
- removed net N$21: J1.B5, J2.B5, J3.B5, J4.B5, J5.B5, J6.B5, J7.B5, J8.B5
- removed net N$22: J1.B6, J2.B6, J3.B6, J4.B6, J5.B6, J6.B6, J7.B6, J8.B6
- removed net N$23: J1.B7, J2.B7, J3.B7, J4.B7, J5.B7, J6.B7, J7.B7, J8.B7
- removed net N$3: J1.A3, J2.A3, J3.A3, J4.A3, J5.A3, J6.A3, J7.A3, J8.A3
- removed net N$33: J1.C1, J2.C1, J3.C1, J4.C1, J5.C1, J6.C1, J7.C1, J8.C1
- removed net N$34: J1.C2, J2.C2, J3.C2, J4.C2, J5.C2, J6.C2, J7.C2, J8.C2
- removed net N$35: J1.C3, J2.C3, J3.C3, J4.C3, J5.C3, J6.C3, J7.C3, J8.C3
- removed net N$36: J1.C4, J2.C4, J3.C4, J4.C4, J5.C4, J6.C4, J7.C4, J8.C4
- removed net N$37: J1.C5, J2.C5, J3.C5, J4.C5, J5.C5, J6.C5, J7.C5, J8.C5
- removed net N$39: J1.C7, J2.C7, J3.C7, J4.C7, J5.C7, J6.C7, J7.C7, J8.C7
- removed net N$4: J1.A4, J2.A4, J3.A4, J4.A4, J5.A4, J6.A4, J7.A4, J8.A4
- removed net N$5: J1.A5, J2.A5, J3.A5, J4.A5, J5.A5, J6.A5, J7.A5, J8.A5
- removed net N$6: J1.A6, J2.A6, J3.A6, J4.A6, J5.A6, J6.A6, J7.A6, J8.A6
- removed net N$7: J1.A7, J2.A7, J3.A7, J4.A7, J5.A7, J6.A7, J7.A7, J8.A7
- new net 24V/12V: J1.A5, J1.A6, J1.B4, J1.B5, J1.B6, J1.C4, J1.C5, J2.A5, J2.A6, J2.B4, J2.B5, J2.B6, J2.C4, J2.C5, J3.A5, J3.A6, J3.B4, J3.B5, J3.B6, J3.C4, J3.C5, J4.A5, J4.A6, J4.B4, J4.B5, J4.B6, J4.C4, J4.C5, J5.A5, J5.A6, J5.B4, J5.B5, J5.B6, J5.C4, J5.C5, J6.A5, J6.A6, J6.B4, J6.B5, J6.B6, J6.C4, J6.C5, J7.A5, J7.A6, J7.B4, J7.B5, J7.B6, J7.C4, J7.C5, J8.A5, J8.A6, J8.B4, J8.B5, J8.B6, J8.C4, J8.C5
- new net 5V: J1.A7, J1.B7, J1.C7, J2.A7, J2.B7, J2.C7, J3.A7, J3.B7, J3.C7, J4.A7, J4.B7, J4.C7, J5.A7, J5.B7, J5.C7, J6.A7, J6.B7, J6.C7, J7.A7, J7.B7, J7.C7, J8.A7, J8.B7, J8.C7
- new net GND: J1.A1, J1.A2, J1.A3, J1.A4, J1.B1, J1.B2, J1.B3, J1.C1, J1.C2, J1.C3, J2.A1, J2.A2, J2.A3, J2.A4, J2.B1, J2.B2, J2.B3, J2.C1, J2.C2, J2.C3, J3.A1, J3.A2, J3.A3, J3.A4, J3.B1, J3.B2, J3.B3, J3.C1, J3.C2, J3.C3, J4.A1, J4.A2, J4.A3, J4.A4, J4.B1, J4.B2, J4.B3, J4.C1, J4.C2, J4.C3, J5.A1, J5.A2, J5.A3, J5.A4, J5.B1, J5.B2, J5.B3, J5.C1, J5.C2, J5.C3, J6.A1, J6.A2, J6.A3, J6.A4, J6.B1, J6.B2, J6.B3, J6.C1, J6.C2, J6.C3, J7.A1, J7.A2, J7.A3, J7.A4, J7.B1, J7.B2, J7.B3, J7.C1, J7.C2, J7.C3, J8.A1, J8.A2, J8.A3, J8.A4, J8.B1, J8.B2, J8.B3, J8.C1, J8.C2, J8.C3
Routing:
- net 3.3V: track 0.00 -> 266.4 mm
- net EXT_7: track 0.00 -> 148.6 mm
- net SS_8: track 0.00 -> 148.4 mm
- net SS_1: track 0.00 -> 148.3 mm
- net SS_2: track 0.00 -> 148.3 mm
- net SS_7: track 0.00 -> 148.3 mm
- net EXT_2: track 0.00 -> 148.2 mm
- net SS_6: track 0.00 -> 148.2 mm
- net SS_9: track 0.00 -> 148.2 mm
- net SS_5: track 0.00 -> 148.2 mm
- net SS_4: track 0.00 -> 148.2 mm
- net SS_3: track 0.00 -> 148.2 mm
- net SS_14: track 0.00 -> 148.2 mm
- net SS_13: track 0.00 -> 148.2 mm
- net SS_12: track 0.00 -> 148.2 mm
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- added copper zone on layer 1, net 24V/12V
- added copper zone on layer 1, net GND
Other:
- board size 170 x 80 mm -> 185 x 80 mm

Commit message: finished backplane
Parts:
- added C1, C3: 10Uf, rc-master-smd:C3216/T
- added C2, C4: 10Uf, rc-master-smd:C1206
- added JP2: (no value), pinhead:2X15
- added U1: LM1084IS-5.0, LM1084IS-5.0:TO254P1435X457-3N
- added U2: LM1084IS-3.3, LM1084IS-5.0:TO254P1435X457-3N
- added XS1: (no value), con-dg55:DG55CB-2P-1
- moved J1 7.00 mm to (25.0, 59.0)
- moved J2 7.00 mm to (45.3, 59.0)
- moved J3 7.00 mm to (65.6, 59.0)
- moved J4 7.00 mm to (86.0, 59.0)
- moved J5 7.00 mm to (106.3, 59.0)
- moved J6 7.00 mm to (126.6, 59.0)
- moved J7 7.00 mm to (146.9, 59.0)
- moved J8 7.00 mm to (167.2, 59.0)
Connections:
- new net N$1: C3.+, U2.3
- new net N$2: C1.+, U1.3
- net 24V/12V: now also XS1.2
- net 3.3V: now also C4.2, JP2.5, U2.2, U2.4
- net 5V: now also C2.2, JP2.3, U1.2, U1.4
- net EXT_1: now also JP2.17
- net EXT_2: now also JP2.19
- net EXT_3: now also JP2.21
- net EXT_4: now also JP2.23
- net EXT_5: now also JP2.25
- net EXT_6: now also JP2.27
- net EXT_7: now also JP2.29
- net GND: now also C1.-, C2.1, C3.-, C4.1, JP2.1, U1.1, U2.1, XS1.1
- net MISO: now also JP2.9
- net MOSI: now also JP2.11
- net SCK: now also JP2.7
- net SCL: now also JP2.15
- net SDA: now also JP2.13
- net SS_1: now also JP2.30
- net SS_10: now also JP2.12
- net SS_11: now also JP2.10
- net SS_12: now also JP2.8
- net SS_13: now also JP2.6
- net SS_14: now also JP2.4
- net SS_15: now also JP2.2
- net SS_2: now also JP2.28
- net SS_3: now also JP2.26
- net SS_4: now also JP2.24
- net SS_5: now also JP2.22
- net SS_6: now also JP2.20
- net SS_7: now also JP2.18
- net SS_8: now also JP2.16
- net SS_9: now also JP2.14
Routing:
- net 3.3V: track 266.4 -> 474.3 mm, vias 0 -> 1
- net GND: track 20.3 -> 182.5 mm, vias 0 -> 1
- net 5V: track 147.3 -> 215.8 mm, vias 0 -> 2
- net EXT_7: track 148.6 -> 207.8 mm, vias 0 -> 1
- net SCK: track 148.2 -> 190.0 mm
- net EXT_4: track 148.2 -> 189.3 mm, vias 0 -> 2
- net SS_10: track 148.2 -> 186.4 mm
- net EXT_6: track 148.2 -> 185.4 mm, vias 0 -> 4
- net SS_9: track 148.2 -> 185.4 mm
- net MISO: track 148.2 -> 182.8 mm
- net EXT_2: track 148.2 -> 181.8 mm, vias 0 -> 2
- net SS_8: track 148.4 -> 181.7 mm, vias 0 -> 1
- net EXT_3: track 148.2 -> 180.8 mm, vias 0 -> 2
- net EXT_1: track 148.2 -> 177.4 mm, vias 0 -> 2
- net EXT_5: track 148.2 -> 176.7 mm, vias 0 -> 2
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Other:
- board size 185 x 80 mm -> 192 x 80 mm
