File: oxygen sensing/oxygen sensing.brd (EAGLE design)
At the start: 100 x 80 mm, 9 parts, among them J1 8-1393644-0, J2 MJ-3536N, J3 MJ-3536N, U1 TLV2333IDGKR

Commit message: general update of most things
Parts:
- added P1: (no value), pinhead:1X01
- added SJ1: SOLDERJUMPERTRACE, SparkFun-Passives:SJ_2S-TRACE
Connections:
- new net N$3: P1.1, SJ1.2
- net SS_5: now also SJ1.1
Changed lines of the file:
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@@
 <attribute name="VALUE" x="96.24633125" y="22.773409375" size="1.27251875" layer="27" rot="R180"/>
+</element>
+<element name="P1" library="pinhead" library_urn="urn:adsk.eagle:library:325" package="1X01" package3d_urn="urn:adsk.eagle:package:22485/2" value="" x="18.3" y="-6.7" locked="yes" smashed="yes">
+<attribute name="NAME" x="19.9538" y="-7.2712" locked="yes" size="1.27" layer="25" ratio="10"/>
+<attribute name="POPULARITY" value="64" x="18.3" y="-6.7" locked="yes" size="1.778" layer="27" display="off"/>
+<attribute name="VALUE" x="17.03" y="-9.875" locked="yes" size="1.27" layer="27"/>
+</element>
+<element name="SJ1" library="SparkFun-Passives" package="SJ_2S-TRACE" value="SOLDERJUMPERTRACE" x="15" y="-7" locked="yes" smashed="yes">
+<attribute name="NAME" x="14.0475" y="-5.73" locked="yes" size="0.4064" layer="25"/>
+<attribute name="VALUE" x="14.0475" y="-8.651" locked="yes" size="0.4064" layer="27"/>
 </element>
 </elements>
@@
 <contactref element="J1" pad="12"/>
 <contactref element="U$1" pad="13"/>
-<wire x1="-2.375" y1="-9.0822" x2="5.6" y2="48.94" width="0" layer="19" extent="1-1"/>
+<contactref element="SJ1" pad="1"/>
+<wire x1="14.492" y1="-7" x2="5.6" y2="48.94" width="0" layer="19" extent="1-1"/>
+<wire x1="-2.375" y1="-9.0822" x2="14.492" y2="-7" width="0" layer="19" extent="1-1"/>
 </signal>
 <signal name="SS_6">
@@
 <wire x1="-2.375" y1="-14.9178" x2="93.6" y2="16" width="0" layer="19" extent="1-1"/>
 <wire x1="-2.85" y1="-4.975" x2="-2.375" y2="-14.9178" width="0" layer="19" extent="1-1"/>
+</signal>
+<signal name="N$3">
+<contactref element="P1" pad="1"/>
+<contactref element="SJ1" pad="2"/>
+<wire x1="15.508" y1="-7" x2="18.3" y2="-6.7" width="0" layer="19" extent="1-1"/>
 </signal>
 </signals>
@@
 </drawing>
 <compatibility>
+<note version="8.2" severity="warning">
+Since Version 8.2, EAGLE supports online libraries. The ids
+of those online libraries will not be understood (or retained)
+with this version.
+</note>
 <note version="8.3" severity="warning">
 Since Version 8.3, EAGLE supports URNs for individual library
@@
 will not be understood (or retained) with this version.
 </note>
+<note version="8.3" severity="warning">
+Since Version 8.3, EAGLE supports the association of 3D packages
+with devices in libraries, schematics, and board files. Those 3D
+packages will not be understood (or retained) with this version.
+</note>
 </compatibility>
