File: oxygen sensing/oxygen sensing.sch (EAGLE design)
At the start: 9 parts, among them J1 8-1393644-0, J2 MJ-3536N, J3 MJ-3536N, U1 TLV2333IDGKR

Commit message: general update of most things
Parts:
- added P1: (no value), pinhead:PINHD-1X1
- added SJ1: SOLDERJUMPERTRACE, SparkFun-Passives:SOLDERJUMPERTRACE
Connections:
- new net N$3: P1.1, SJ1.2
- net SS_5: now also SJ1.1
Other:
- moved on the sheet: J1
