File: prototype card/prototype card.brd (EAGLE design)
At the start: 100 x 80 mm, 6 parts, among them J1 8-1393644-0

Commit message: general update of most things
Parts:
- added J2: TBP02R1-381-14BE, TBP02R1-381-14BE:CUI_TBP02R1-381-14BE
Routing:
- net MISO: track 0.00 -> 34.2 mm, vias 0 -> 1
- net SS_1: track 0.00 -> 33.5 mm, vias 0 -> 1
- net SS_2: track 0.00 -> 33.3 mm, vias 0 -> 1
- net SS_7: track 0.00 -> 33.1 mm
- net SS_5: track 0.00 -> 32.9 mm, vias 0 -> 1
- net SS_6: track 0.00 -> 31.9 mm
- net SCK: track 0.00 -> 31.6 mm, vias 0 -> 1
- net SS_4: track 0.00 -> 30.4 mm
- net SS_3: track 0.00 -> 29.1 mm, vias 0 -> 1
- net MOSI: track 0.00 -> 25.0 mm, vias 0 -> 1
- net SDA: track 0.00 -> 21.4 mm, vias 0 -> 1
- net SS_13: track 0.00 -> 16.2 mm
- net SS_9: track 0.00 -> 16.2 mm
- net SS_14: track 0.00 -> 15.8 mm
- net SS_12: track 0.00 -> 15.4 mm
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
Commit message: fixed library attributes for the din41612 connector, fixed git problems
Parts:
- J1: value 8-1393644-0 -> 09231486921; device 8-1393644-0:TE_8-1393644-0 -> din41612_48_pin_board:HARTING_09231486921
Changed lines of the file:
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@@
 <drawing>
 <settings>
-<setting alwaysvectorfont="yes"/>
+<setting alwaysvectorfont="no"/>
 <setting verticaltext="up"/>
 </settings>
@@
 SS_1
 </text>
-<hole x="25.27" y="13.98" drill="0.8" grouprefs="22_PADS PAD"/>
-<rectangle x1="24.27" y1="12.98" x2="26.27" y2="14.98" layer="17" grouprefs="22_PADS PAD"/>
+<hole x="25.27" y="13.98" drill="0.8" grouprefs="PAD 22_PADS"/>
+<rectangle x1="24.27" y1="12.98" x2="26.27" y2="14.98" layer="17" grouprefs="PAD 22_PADS"/>
 <hole x="25.27" y="13.98" drill="0.8" grouprefs="22_PADS"/>
 <hole x="27.81" y="13.98" drill="0.8" grouprefs="22_PADS"/>
@@
 </groups>
 <elements>
-<element name="J1" library="8-1393644-0" package="TE_8-1393644-0" value="8-1393644-0" x="5.6" y="21" smashed="yes" rot="R270">
+<element name="J1" library="din41612_48_pin_board" package="HARTING_09231486921" value="09231486921" x="5.6" y="21" smashed="yes" rot="R270">
 <attribute name="AVAILABILITY" value="In Stock" x="5.6" y="21" size="1.778" layer="27" rot="R270" display="off"/>
-<attribute name="COMMENT" value="8-1393644-0" x="5.6" y="21" size="1.778" layer="27" rot="R270" display="off"/>
+<attribute name="COMMENT" value="09231486921" x="5.6" y="21" size="1.778" layer="27" rot="R270" display="off"/>
 <attribute name="DESCRIPTION" value=" Conn DIN 41612 M 48 POS 2.54mm Solder RA Thru-Hole Tray " x="5.6" y="21" size="1.778" layer="27" rot="R270" display="off"/>
 <attribute name="EU_ROHS_COMPLIANCE" value="Compliant" x="5.6" y="21" size="1.778" layer="27" rot="R270" display="off"/>
-<attribute name="MF" value="TE Connectivity" x="5.6" y="21" size="1.778" layer="27" rot="R270" display="off"/>
-<attribute name="MP" value="8-1393644-0" x="5.6" y="21" size="1.778" layer="27" rot="R270" display="off"/>
+<attribute name="MF" value="HARTING" x="5.6" y="21" size="1.778" layer="27" rot="R270" display="off"/>
+<attribute name="MP" value="09231486921" x="5.6" y="21" size="1.778" layer="27" rot="R270" display="off"/>
 <attribute name="NAME" x="12.605" y="67.73" size="1.27" layer="25" rot="R270"/>
 <attribute name="PACKAGE" value="None" x="5.6" y="21" size="1.778" layer="27" rot="R270" display="off"/>
-<attribute name="PRICE" value="None" x="5.6" y="21" size="1.778" layer="27" rot="R270" display="off"/>
-<attribute name="PURCHASE-URL" value="https://pricing.snapeda.com/search/part/8-1393644-0/?ref=eda" x="5.6" y="21" size="1.778" layer="27" rot="R270" display="off"/>
+<attribute name="PRICE" value="6$" x="5.6" y="21" size="1.778" layer="27" rot="R270" display="off"/>
+<attribute name="PURCHASE-URL-DIGIKEY" value="https://www.digikey.ca/en/products/detail/harting/09231486921/3180439" x="5.6" y="21" size="1.778" layer="27" rot="R270" display="off"/>
 <attribute name="VALUE" x="-8.59" y="67.73" size="1.27" layer="27" rot="R270"/>
 </element>
