File: prototype card/prototype card.brd (EAGLE design)
At the start: 100 x 80 mm, 22 parts, among them J1 09231486921, J2 TBP02R1-381-14BE

Commit message: updated libraries to generate better bom's
Routing:
- net 24V/12V: track 125.7 -> 126.8 mm
Changed lines of the file:
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@@
 CS_1
 </text>
-<hole x="25.27" y="13.75" drill="0.8" grouprefs="PAD 22_PADS"/>
-<rectangle x1="24.27" y1="12.75" x2="26.27" y2="14.75" layer="17" grouprefs="PAD 22_PADS"/>
+<hole x="25.27" y="13.75" drill="0.8" grouprefs="22_PADS PAD"/>
+<rectangle x1="24.27" y1="12.75" x2="26.27" y2="14.75" layer="17" grouprefs="22_PADS PAD"/>
 <hole x="27.81" y="13.75" drill="0.8" grouprefs="22_PADS"/>
 <hole x="30.35" y="13.75" drill="0.8" grouprefs="22_PADS"/>
@@
 </groups>
 <elements>
-<element name="J1" library="din41612_48_pin_board" package="HARTING_09231486921" value="09231486921" x="5.6" y="20.95" smashed="yes" rot="R270">
-<attribute name="AVAILABILITY" value="In Stock" x="5.6" y="20.95" size="1.778" layer="27" rot="R270" display="off"/>
-<attribute name="COMMENT" value="09231486921" x="5.6" y="20.95" size="1.778" layer="27" rot="R270" display="off"/>
-<attribute name="DESCRIPTION" value=" Conn DIN 41612 M 48 POS 2.54mm Solder RA Thru-Hole Tray " x="5.6" y="20.95" size="1.778" layer="27" rot="R270" display="off"/>
-<attribute name="EU_ROHS_COMPLIANCE" value="Compliant" x="5.6" y="20.95" size="1.778" layer="27" rot="R270" display="off"/>
-<attribute name="MF" value="HARTING" x="5.6" y="20.95" size="1.778" layer="27" rot="R270" display="off"/>
-<attribute name="MP" value="09231486921" x="5.6" y="20.95" size="1.778" layer="27" rot="R270" display="off"/>
+<element name="J1" library="din41612_48_pin_board" package="HARTING_09231486921" package3d_urn="urn:adsk.eagle:package:31078162/1" value="09231486921" x="5.6" y="20.95" smashed="yes" rot="R270">
+<attribute name="MANUFACTURER-PART-NUMBER" value="09231486921" x="5.6" y="20.95" size="1.778" layer="27" rot="R270" display="off"/>
 <attribute name="NAME" x="2.605" y="11.68" size="1.27" layer="25"/>
 <attribute name="PACKAGE" value="None" x="5.6" y="20.95" size="1.778" layer="27" rot="R270" display="off"/>
-<attribute name="PRICE" value="6$" x="5.6" y="20.95" size="1.778" layer="27" rot="R270" display="off"/>
-<attribute name="PURCHASE-URL-DIGIKEY" value="https://www.digikey.ca/en/products/detail/harting/09231486921/3180439" x="5.6" y="20.95" size="1.778" layer="27" rot="R270" display="off"/>
+<attribute name="SIMILAR-COMPONENTS" value="" x="5.6" y="20.95" size="1.778" layer="27" rot="R270" display="off"/>
 <attribute name="VALUE" x="-8.59" y="67.68" size="1.27" layer="27" rot="R270"/>
 </element>
@@
 </element>
 <element name="J2" library="TBP02R1-381-14BE" package="CUI_TBP02R1-381-14BE" value="TBP02R1-381-14BE" x="95" y="64.765" smashed="yes" rot="R270">
-<attribute name="AVAILABILITY" value="In Stock" x="95" y="64.765" size="1.778" layer="27" rot="R270" display="off"/>
-<attribute name="CUI_PURCHASE_URL" value="https://www.cuidevices.com/product/interconnect/connectors/terminal-blocks/tbp02r1-381-series?utm_source=snapeda.com&amp;utm_medium=referral&amp;utm_campaign=snapedaBOM" x="95" y="64.765" size="1.778" layer="27" rot="R270" display="off"/>
-<attribute name="DESCRIPTION" value="2~24 Poles, Pluggable,Receptacle, Horizontal, 3.81 Pitch, Terminal Block Connector" x="95" y="64.765" size="1.778" layer="27" rot="R270" display="off"/>
-<attribute name="MF" value="CUI Devices" x="95" y="64.765" size="1.778" layer="27" rot="R270" display="off"/>
-<attribute name="MP" value="TBP02R1-381-14BE" x="95" y="64.765" size="1.778" layer="27" rot="R270" display="off"/>
+<attribute name="MANUFACTURER-PART-NUMBER" value="TBP02R1-381-14BE" x="95" y="64.765" size="1.778" layer="27" rot="R270" display="off"/>
 <attribute name="PACKAGE" value="None" x="95" y="64.765" size="1.778" layer="27" rot="R270" display="off"/>
-<attribute name="PRICE" value="None" x="95" y="64.765" size="1.778" layer="27" rot="R270" display="off"/>
-<attribute name="PURCHASE-URL" value="https://pricing.snapeda.com/search/part/TBP02R1-381-14BE/?ref=eda" x="95" y="64.765" size="1.778" layer="27" rot="R270" display="off"/>
+<attribute name="SIMILAR-COMPONENTS" value="" x="95" y="64.765" size="1.778" layer="27" rot="R270" display="off"/>
 </element>
 <element name="J4" library="SparkFun-Connectors" package="1X01_LONGPAD" value="" x="91.28" y="15.25" smashed="yes" rot="R90">
@@
 <contactref element="JP5" pad="28"/>
 <contactref element="JP5" pad="29"/>
-<wire x1="91.83" y1="6" x2="14" y2="6" width="4" layer="1"/>
+<wire x1="91.83" y1="6" x2="14" y2="6" width="3.8" layer="1"/>
 <wire x1="14" y1="6" x2="8.14" y2="11.86" width="5" layer="1"/>
 <wire x1="8.14" y1="11.86" x2="8.14" y2="20.95" width="5" layer="1"/>
@@
 <contactref element="JP2" pad="28"/>
 <contactref element="JP2" pad="29"/>
-<wire x1="91.83" y1="10" x2="87.83" y2="10" width="5" layer="16"/>
-<wire x1="87.83" y1="10" x2="18.17" y2="10" width="4" layer="16"/>
+<wire x1="87.83" y1="10" x2="18.17" y2="10" width="3.8" layer="16"/>
 <wire x1="18.17" y1="10" x2="16.17" y2="12" width="4" layer="16"/>
 <wire x1="16.17" y1="12" x2="15.17" y2="12" width="4.6" layer="16"/>
@@
 <wire x1="10.68" y1="28.57" x2="8.14" y2="28.57" width="1.6" layer="16"/>
 <wire x1="8.14" y1="28.57" x2="8.14" y2="31.11" width="1.6" layer="16"/>
-<wire x1="86.75" y1="10" x2="89.29" y2="10" width="0" layer="19" extent="1-1"/>
+<wire x1="86.75" y1="10" x2="89.29" y2="10" width="3.8" layer="16"/>
+<wire x1="89.29" y1="10" x2="91.83" y2="10" width="3.8" layer="16"/>
+<wire x1="87.83" y1="10" x2="86.75" y2="10" width="0" layer="19" extent="16-16"/>
 <wire x1="84.21" y1="10" x2="86.75" y2="10" width="0" layer="19" extent="1-1"/>
 <wire x1="81.67" y1="10" x2="84.21" y2="10" width="0" layer="19" extent="1-1"/>
@@
 <wire x1="25.79" y1="10" x2="28.33" y2="10" width="0" layer="19" extent="1-1"/>
 <wire x1="23.25" y1="10" x2="25.79" y2="10" width="0" layer="19" extent="1-1"/>
-<wire x1="20.71" y1="10" x2="23.25" y2="10" width="0" layer="19" extent="1-1"/>
-<wire x1="91.83" y1="10" x2="89.29" y2="10" width="0" layer="19" extent="1-1"/>
+<wire x1="20.71" y1="10" x2="18.17" y2="10" width="0" layer="19" extent="1-1"/>
 </signal>
 <signal name="5V">

Commit message: finished V2.2 control module update
Other:
- board text added: "PolyVent prototyping board V1.2 - Public Invention -Liscence: CERN OHL V2.0"
- board text removed: "PolyVent prototyping board V1.1 - Public Invention -Liscence: CERN OHL V2.0"
Changed lines of the file:
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@@
 CS_1
 </text>
-<hole x="25.27" y="13.75" drill="0.8" grouprefs="22_PADS PAD"/>
-<rectangle x1="24.27" y1="12.75" x2="26.27" y2="14.75" layer="17" grouprefs="22_PADS PAD"/>
+<hole x="25.27" y="13.75" drill="0.8" grouprefs="PAD 22_PADS"/>
+<rectangle x1="24.27" y1="12.75" x2="26.27" y2="14.75" layer="17" grouprefs="PAD 22_PADS"/>
 <hole x="27.81" y="13.75" drill="0.8" grouprefs="22_PADS"/>
 <hole x="30.35" y="13.75" drill="0.8" grouprefs="22_PADS"/>
@@
 <rectangle x1="24" y1="12" x2="87.49" y2="63.4" layer="30"/>
 <rectangle x1="24" y1="12" x2="87.49" y2="63.4" layer="29"/>
-<text x="7" y="77" size="1.778" layer="29">PolyVent prototyping board V1.1 - Public Invention -Liscence: CERN OHL V2.0</text>
+<text x="7" y="77" size="1.778" layer="29">PolyVent prototyping board V1.2 - Public Invention -Liscence: CERN OHL V2.0</text>
 <text x="16.81" y="3.12" size="2" layer="29" distance="0" align="bottom-right">24V/12V
 GND
