File: prototype card/prototype card.sch (EAGLE design)
At the start: 6 parts, among them J1 8-1393644-0

Commit message: general update of most things
Parts:
- added J2: TBP02R1-381-14BE, TBP02R1-381-14BE:TBP02R1-381-14BE
Changed lines of the file:
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@@
 <part name="JP4" library="pinhead" library_urn="urn:adsk.eagle:library:325" deviceset="PINHD-1X30" device="" package3d_urn="urn:adsk.eagle:package:22460/2"/>
 <part name="JP5" library="pinhead" library_urn="urn:adsk.eagle:library:325" deviceset="PINHD-1X30" device="" package3d_urn="urn:adsk.eagle:package:22460/2"/>
+<part name="J2" library="TBP02R1-381-14BE" deviceset="TBP02R1-381-14BE" device=""/>
 </parts>
 <sheets>
@@
 <attribute name="NAME" x="-54.61" y="92.075" size="1.778" layer="95"/>
 <attribute name="VALUE" x="-54.61" y="10.16" size="1.778" layer="96"/>
+</instance>
+<instance part="J2" gate="G$1" x="-127" y="116.84" smashed="yes">
+<attribute name="NAME" x="-132.58" y="137.16" size="1.778" layer="95"/>
+<attribute name="VALUE" x="-132.08" y="96.52" size="1.778" layer="96"/>
 </instance>
 </instances>
@@
 </segment>
 </net>
+<net name="N$3" class="0">
+</net>
 </nets>

Commit message: fixed library attributes for the din41612 connector, fixed git problems
Parts:
- J1: value 8-1393644-0 -> 09231486921; device 8-1393644-0:8-1393644-0 -> din41612_48_pin_board:09231486921
Changed lines of the file:
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@@
 </classes>
 <parts>
-<part name="J1" library="8-1393644-0" deviceset="8-1393644-0" device=""/>
+<part name="J1" library="din41612_48_pin_board" deviceset="09231486921" device=""/>
 <part name="GND1" library="supply1" library_urn="urn:adsk.eagle:library:371" deviceset="GND" device=""/>
 <part name="GND2" library="supply1" library_urn="urn:adsk.eagle:library:371" deviceset="GND" device=""/>
