File: motor control card/motor control board.sch (EAGLE design)
At the start: 13 parts, among them J1 8-1393644-0, J2 TBP02R1-381-07BE, J3 TBP02R1-381-07BE

Commit message: fixed library attributes for the din41612 connector, fixed git problems
Parts:
- J1: value 8-1393644-0 -> 09231486921; device 8-1393644-0:8-1393644-0 -> din41612_48_pin_board:09231486921
Changed lines of the file:
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@@
 </classes>
 <parts>
-<part name="J1" library="8-1393644-0" deviceset="8-1393644-0" device=""/>
+<part name="J1" library="din41612_48_pin_board" deviceset="09231486921" device=""/>
 <part name="GND1" library="supply1" library_urn="urn:adsk.eagle:library:371" deviceset="GND" device=""/>
 <part name="GND2" library="supply1" library_urn="urn:adsk.eagle:library:371" deviceset="GND" device=""/>

Commit message: added cam data
Parts:
- U$1, U$2: device high power stepper driver 36V4:POLOLU_HIGH-POWER_STEPPER_MOTOR_DRIVER_36V4 -> high_power_stepper_driver_36V4:POLOLU_HIGH-POWER_STEPPER_MOTOR_DRIVER_36V4
Changed lines of the file:
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@@
 <part name="GND2" library="supply1" library_urn="urn:adsk.eagle:library:371" deviceset="GND" device=""/>
 <part name="GND3" library="supply1" library_urn="urn:adsk.eagle:library:371" deviceset="GND" device=""/>
-<part name="U$1" library="high power stepper driver 36V4" deviceset="POLOLU_HIGH-POWER_STEPPER_MOTOR_DRIVER_36V4" device=""/>
+<part name="U$1" library="high_power_stepper_driver_36V4" deviceset="POLOLU_HIGH-POWER_STEPPER_MOTOR_DRIVER_36V4" device=""/>
 <part name="U$3" library="SparkFun-SAMD21-Mini-Breakout" deviceset="SAM_D21_MINI_BREAKOUT" device=""/>
 <part name="GND5" library="supply1" library_urn="urn:adsk.eagle:library:371" deviceset="GND" device=""/>
-<part name="U$2" library="high power stepper driver 36V4" deviceset="POLOLU_HIGH-POWER_STEPPER_MOTOR_DRIVER_36V4" device=""/>
+<part name="U$2" library="high_power_stepper_driver_36V4" deviceset="POLOLU_HIGH-POWER_STEPPER_MOTOR_DRIVER_36V4" device=""/>
 <part name="J2" library="TBP02R1-381-07BE" deviceset="TBP02R1-381-07BE" device=""/>
 <part name="GND6" library="supply1" library_urn="urn:adsk.eagle:library:371" deviceset="GND" device=""/>
