File: motor control card/motor control board.sch (EAGLE design)
At the start: 13 parts, among them J1 09231486921, J2 TBP02R1-381-07BE, J3 TBP02R1-381-07BE

Commit message: re routed broken connections from last commit, parts should work now
Connections:
- net GND: now also U$3.GND2; no longer U$3.AREF
Changed lines of the file:
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@@
 </segment>
 <segment>
-<pinref part="U$3" gate="G$1" pin="AREF"/>
+<pinref part="U$3" gate="G$1" pin="GND2"/>
 <pinref part="GND9" gate="1" pin="GND"/>
-<wire x1="25.4" y1="190.5" x2="53.34" y2="190.5" width="0.1524" layer="91"/>
+<wire x1="25.4" y1="195.58" x2="53.34" y2="195.58" width="0.1524" layer="91"/>
+<wire x1="53.34" y1="195.58" x2="53.34" y2="190.5" width="0.1524" layer="91"/>
 </segment>
 </net>

Commit message: improved silkscreen for valve board
Connections:
- net SS_1 renamed CS_1
- net SS_10 renamed CS_10
- net SS_11 renamed CS_11
- net SS_12 renamed CS_12
- net SS_13 renamed CS_13
- net SS_14 renamed CS_14
- net SS_15 renamed CS_15
- net SS_2 renamed CS_2
- net SS_3 renamed CS_3
- net SS_4 renamed CS_4
- net SS_5 renamed CS_5
- net SS_6 renamed CS_6
- net SS_7 renamed CS_7
- net SS_8 renamed CS_8
- net SS_9 renamed CS_9
Changed lines of the file:
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@@
 </segment>
 </net>
-<net name="SS_1" class="0">
+<net name="CS_1" class="0">
 <segment>
 <pinref part="J1" gate="G$1" pin="8"/>
@@
 </segment>
 </net>
-<net name="SS_2" class="0">
+<net name="CS_2" class="0">
 <segment>
 <pinref part="J1" gate="G$1" pin="9"/>
@@
 </segment>
 </net>
-<net name="SS_3" class="0">
+<net name="CS_3" class="0">
 <segment>
 <pinref part="J1" gate="G$1" pin="10"/>
@@
 </segment>
 </net>
-<net name="SS_4" class="0">
+<net name="CS_4" class="0">
 <segment>
 <pinref part="J1" gate="G$1" pin="11"/>
@@
 </segment>
 </net>
-<net name="SS_5" class="0">
+<net name="CS_5" class="0">
 <segment>
 <pinref part="J1" gate="G$1" pin="12"/>
@@
 </segment>
 </net>
-<net name="SS_6" class="0">
+<net name="CS_6" class="0">
 <segment>
 <pinref part="J1" gate="G$1" pin="13"/>
@@
 </segment>
 </net>
-<net name="SS_7" class="0">
+<net name="CS_7" class="0">
 <segment>
 <pinref part="J1" gate="G$1" pin="14"/>
@@
 </segment>
 </net>
-<net name="SS_8" class="0">
+<net name="CS_8" class="0">
 <segment>
 <pinref part="J1" gate="G$1" pin="24"/>
@@
 </segment>
 </net>
-<net name="SS_9" class="0">
+<net name="CS_9" class="0">
 <segment>
 <pinref part="J1" gate="G$1" pin="25"/>
@@
 </segment>
 </net>
-<net name="SS_10" class="0">
+<net name="CS_10" class="0">
 <segment>
 <pinref part="J1" gate="G$1" pin="26"/>
@@
 </segment>
 </net>
-<net name="SS_11" class="0">
+<net name="CS_11" class="0">
 <segment>
 <pinref part="J1" gate="G$1" pin="27"/>
@@
 </segment>
 </net>
-<net name="SS_12" class="0">
+<net name="CS_12" class="0">
 <segment>
 <pinref part="J1" gate="G$1" pin="28"/>
@@
 </segment>
 </net>
-<net name="SS_13" class="0">
+<net name="CS_13" class="0">
 <segment>
 <pinref part="J1" gate="G$1" pin="29"/>
@@
 </segment>
 </net>
-<net name="SS_14" class="0">
+<net name="CS_14" class="0">
 <segment>
 <pinref part="J1" gate="G$1" pin="30"/>
@@
 </segment>
 </net>
-<net name="SS_15" class="0">
+<net name="CS_15" class="0">
 <segment>
 <pinref part="J1" gate="G$1" pin="45"/>
