File: motor control card/motor control board.sch (EAGLE design)
At the start: 18 parts, among them J1 09231486921, J2 TBP02R1-381-07BE, J3 TBP02R1-381-07BE

Commit message: updated libraries to generate better bom's
Parts:
- U$4: value (none) -> SAM_D21_MINI_BREAKOUT
Changed lines of the file:
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@@
 </classes>
 <parts>
-<part name="J1" library="din41612_48_pin_board" deviceset="09231486921" device=""/>
+<part name="J1" library="din41612_48_pin_board" deviceset="09231486921" device="" package3d_urn="urn:adsk.eagle:package:31078162/1"/>
 <part name="GND1" library="supply1" library_urn="urn:adsk.eagle:library:371" deviceset="GND" device=""/>
 <part name="GND2" library="supply1" library_urn="urn:adsk.eagle:library:371" deviceset="GND" device=""/>
@@
 <part name="P2" library="pinhead" library_urn="urn:adsk.eagle:library:325" deviceset="PINHD-1X1" device="" package3d_urn="urn:adsk.eagle:package:22485/2"/>
 <part name="P1" library="pinhead" library_urn="urn:adsk.eagle:library:325" deviceset="PINHD-1X1" device="" package3d_urn="urn:adsk.eagle:package:22485/2"/>
-<part name="SJ1" library="SparkFun-Passives" deviceset="SOLDERJUMPER" device="TRACE"/>
-<part name="SJ2" library="SparkFun-Passives" deviceset="SOLDERJUMPER" device="TRACE"/>
+<part name="SJ1" library="SparkFun-Passives" deviceset="SOLDERJUMPER" device="TRACE" package3d_urn="urn:adsk.eagle:package:30824525/1"/>
+<part name="SJ2" library="SparkFun-Passives" deviceset="SOLDERJUMPER" device="TRACE" package3d_urn="urn:adsk.eagle:package:30824525/1"/>
 <part name="P3" library="pinhead" library_urn="urn:adsk.eagle:library:325" deviceset="PINHD-1X1" device="" package3d_urn="urn:adsk.eagle:package:22485/2"/>
-<part name="SJ3" library="SparkFun-Passives" deviceset="SOLDERJUMPER" device="TRACE"/>
+<part name="SJ3" library="SparkFun-Passives" deviceset="SOLDERJUMPER" device="TRACE" package3d_urn="urn:adsk.eagle:package:30824525/1"/>
 <part name="JP1" library="pinhead" library_urn="urn:adsk.eagle:library:325" deviceset="PINHD-1X15" device="" package3d_urn="urn:adsk.eagle:package:22424/2"/>
 <part name="J3" library="TBP02R1-381-07BE" deviceset="TBP02R1-381-07BE" device=""/>
@@
 <part name="GND4" library="supply1" library_urn="urn:adsk.eagle:library:371" deviceset="GND" device=""/>
 <part name="GND9" library="supply1" library_urn="urn:adsk.eagle:library:371" deviceset="GND" device=""/>
-<part name="SJ4" library="SparkFun-Passives" deviceset="SOLDERJUMPER" device="TRACE"/>
-<part name="SJ5" library="SparkFun-Passives" deviceset="SOLDERJUMPER" device="TRACE"/>
+<part name="SJ4" library="SparkFun-Passives" deviceset="SOLDERJUMPER" device="TRACE" package3d_urn="urn:adsk.eagle:package:30824525/1"/>
+<part name="SJ5" library="SparkFun-Passives" deviceset="SOLDERJUMPER" device="TRACE" package3d_urn="urn:adsk.eagle:package:30824525/1"/>
 <part name="U$4" library="SparkFun-SAMD21-Mini-Breakout" deviceset="SAM_D21_MINI_BREAKOUT" device=""/>
 <part name="JP5" library="pinhead" library_urn="urn:adsk.eagle:library:325" deviceset="PINHD-1X4" device="" package3d_urn="urn:adsk.eagle:package:22407/2"/>

Commit message: finished V2.2 control module update
Other:
- note added: "Connectors"
- note added: "Microcontroller"
- note added: "Motor Drivers"
- note added: "Not Working Nov 24, 2021"
- moved on the sheet: J1, J2, J3, JP1, JP5, JP6, JP7, P1, P2, P3, SJ1, SJ2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
