File: sensor card/sensor card.brd (EAGLE design)
At the start: 100 x 80 mm, 21 parts, among them J1 8-1393644-0, J2 MJ-3536N, J3 MJ-3536N, X1 S4B-XH-A, X2 S4B-XH-A

Commit message: fixed library attributes for the din41612 connector, fixed git problems
Parts:
- J1: value 8-1393644-0 -> 09231486921; device 8-1393644-0:TE_8-1393644-0 -> din41612_48_pin_board:HARTING_09231486921
Changed lines of the file:
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@@
 </autorouter>
 <elements>
-<element name="J1" library="8-1393644-0" package="TE_8-1393644-0" value="8-1393644-0" x="5.6" y="21" smashed="yes" rot="R270">
+<element name="J1" library="din41612_48_pin_board" package="HARTING_09231486921" value="09231486921" x="5.6" y="21" smashed="yes" rot="R270">
 <attribute name="AVAILABILITY" value="In Stock" x="5.6" y="21" size="1.778" layer="27" rot="R270" display="off"/>
-<attribute name="COMMENT" value="8-1393644-0" x="5.6" y="21" size="1.778" layer="27" rot="R270" display="off"/>
+<attribute name="COMMENT" value="09231486921" x="5.6" y="21" size="1.778" layer="27" rot="R270" display="off"/>
 <attribute name="DESCRIPTION" value=" Conn DIN 41612 M 48 POS 2.54mm Solder RA Thru-Hole Tray " x="5.6" y="21" size="1.778" layer="27" rot="R270" display="off"/>
 <attribute name="EU_ROHS_COMPLIANCE" value="Compliant" x="5.6" y="21" size="1.778" layer="27" rot="R270" display="off"/>
-<attribute name="MF" value="TE Connectivity" x="5.6" y="21" size="1.778" layer="27" rot="R270" display="off"/>
-<attribute name="MP" value="8-1393644-0" x="5.6" y="21" size="1.778" layer="27" rot="R270" display="off"/>
+<attribute name="MF" value="HARTING" x="5.6" y="21" size="1.778" layer="27" rot="R270" display="off"/>
+<attribute name="MP" value="09231486921" x="5.6" y="21" size="1.778" layer="27" rot="R270" display="off"/>
 <attribute name="NAME" x="12.605" y="67.73" size="1.27" layer="25" rot="R270"/>
 <attribute name="PACKAGE" value="None" x="5.6" y="21" size="1.778" layer="27" rot="R270" display="off"/>
-<attribute name="PRICE" value="None" x="5.6" y="21" size="1.778" layer="27" rot="R270" display="off"/>
-<attribute name="PURCHASE-URL" value="https://pricing.snapeda.com/search/part/8-1393644-0/?ref=eda" x="5.6" y="21" size="1.778" layer="27" rot="R270" display="off"/>
+<attribute name="PRICE" value="6$" x="5.6" y="21" size="1.778" layer="27" rot="R270" display="off"/>
+<attribute name="PURCHASE-URL-DIGIKEY" value="https://www.digikey.ca/en/products/detail/harting/09231486921/3180439" x="5.6" y="21" size="1.778" layer="27" rot="R270" display="off"/>
 <attribute name="VALUE" x="-8.59" y="67.73" size="1.27" layer="27" rot="R270"/>
 </element>
@@
 <vertex x="100" y="80"/>
 </polygon>
+<wire x1="91" y1="34.25" x2="91" y2="47.25" width="0" layer="19" extent="1-1"/>
+<wire x1="82.4" y1="31.2" x2="91" y2="34.25" width="0" layer="19" extent="1-1"/>
+<wire x1="79.9" y1="26" x2="82.4" y2="31.2" width="0" layer="19" extent="1-1"/>
+<wire x1="82.4" y1="19.2" x2="79.9" y2="26" width="0" layer="19" extent="1-1"/>
+<wire x1="79.9" y1="14" x2="82.4" y2="19.2" width="0" layer="19" extent="1-1"/>
+<wire x1="72.125" y1="26.2178" x2="79.9" y2="26" width="0" layer="19" extent="1-1"/>
+<wire x1="71.475" y1="26.2178" x2="72.125" y2="26.2178" width="0" layer="19" extent="1-1"/>
+<wire x1="66.925" y1="26.2178" x2="71.475" y2="26.2178" width="0" layer="19" extent="1-1"/>
+<wire x1="71.475" y1="20.3822" x2="71.475" y2="26.2178" width="0" layer="19" extent="1-1"/>
+<wire x1="72.125" y1="20.3822" x2="71.475" y2="20.3822" width="0" layer="19" extent="1-1"/>
+<wire x1="70.175" y1="20.3822" x2="71.475" y2="20.3822" width="0" layer="19" extent="1-1"/>
+<wire x1="68.875" y1="20.3822" x2="70.175" y2="20.3822" width="0" layer="19" extent="1-1"/>
+<wire x1="67.575" y1="20.3822" x2="68.875" y2="20.3822" width="0" layer="19" extent="1-1"/>
+<wire x1="66.925" y1="20.3822" x2="67.575" y2="20.3822" width="0" layer="19" extent="1-1"/>
+<wire x1="61.81" y1="46.35" x2="66.925" y2="26.2178" width="0" layer="19" extent="1-1"/>
+<wire x1="46.81" y1="56.683334375" x2="61.81" y2="46.35" width="0" layer="19" extent="1-1"/>
+<wire x1="62.81" y1="67.016659375" x2="46.81" y2="56.683334375" width="0" layer="19" extent="1-1"/>
+<wire x1="46.81" y1="77.35" x2="62.81" y2="67.016659375" width="0" layer="19" extent="1-1"/>
+<wire x1="10.68" y1="26.08" x2="46.81" y2="56.683334375" width="0" layer="19" extent="1-1"/>
+<wire x1="10.68" y1="23.54" x2="10.68" y2="26.08" width="0" layer="19" extent="1-1"/>
+<wire x1="8.14" y1="26.08" x2="10.68" y2="26.08" width="0" layer="19" extent="1-1"/>
+<wire x1="5.6" y1="26.08" x2="8.14" y2="26.08" width="0" layer="19" extent="1-1"/>
+<wire x1="5.6" y1="28.62" x2="5.6" y2="26.08" width="0" layer="19" extent="1-1"/>
+<wire x1="10.68" y1="21" x2="10.68" y2="23.54" width="0" layer="19" extent="1-1"/>
+<wire x1="8.14" y1="23.54" x2="10.68" y2="23.54" width="0" layer="19" extent="1-1"/>
+<wire x1="5.6" y1="23.54" x2="5.6" y2="26.08" width="0" layer="19" extent="1-1"/>
+<wire x1="8.14" y1="21" x2="10.68" y2="21" width="0" layer="19" extent="1-1"/>
+<wire x1="5.6" y1="21" x2="5.6" y2="23.54" width="0" layer="19" extent="1-1"/>
 </signal>
 <signal name="5V">

Commit message: added cam data
Parts:
- U$1, U$3, U$4, U$5: value SCCDRRV100MDSA3SSCDRRV100MDSA3 -> SSCDRRV100MDSA3
Changed lines of the file:
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@@
 <attribute name="VALUE" x="-8.59" y="67.73" size="1.27" layer="27" rot="R270"/>
 </element>
-<element name="U$1" library="SCCDRRV100MDSA3" package="DIP1270W53P254L1303H508Q8B" package3d_urn="urn:adsk.eagle:package:23793141/1" value="SCCDRRV100MDSA3SSCDRRV100MDSA3" x="43" y="71" smashed="yes" rot="R270"/>
+<element name="U$1" library="SCCDRRV100MDSA3" package="DIP1270W53P254L1303H508Q8B" package3d_urn="urn:adsk.eagle:package:23793141/1" value="SSCDRRV100MDSA3" x="43" y="71" smashed="yes" rot="R270"/>
 <element name="U$2" library="MCP346XRT-E:ST" package="TSSOP20" value="MCP346X-E/ST" x="69.2" y="23.3" smashed="yes">
 <attribute name="NAME" x="65.6544" y="21.2172" size="1.016" layer="25" ratio="10" rot="R90"/>
@@
 <attribute name="NAME" x="26.0475" y="30.27" size="0.4064" layer="25"/>
 </element>
-<element name="U$3" library="SCCDRRV100MDSA3" package="DIP1270W53P254L1303H508Q8B" package3d_urn="urn:adsk.eagle:package:23793141/1" value="SCCDRRV100MDSA3SSCDRRV100MDSA3" x="59" y="60.666659375" smashed="yes" rot="R270"/>
-<element name="U$4" library="SCCDRRV100MDSA3" package="DIP1270W53P254L1303H508Q8B" package3d_urn="urn:adsk.eagle:package:23793141/1" value="SCCDRRV100MDSA3SSCDRRV100MDSA3" x="43" y="50.333334375" smashed="yes" rot="R270"/>
-<element name="U$5" library="SCCDRRV100MDSA3" package="DIP1270W53P254L1303H508Q8B" package3d_urn="urn:adsk.eagle:package:23793141/1" value="SCCDRRV100MDSA3SSCDRRV100MDSA3" x="58" y="40" smashed="yes" rot="R270"/>
+<element name="U$3" library="SCCDRRV100MDSA3" package="DIP1270W53P254L1303H508Q8B" package3d_urn="urn:adsk.eagle:package:23793141/1" value="SSCDRRV100MDSA3" x="59" y="60.666659375" smashed="yes" rot="R270"/>
+<element name="U$4" library="SCCDRRV100MDSA3" package="DIP1270W53P254L1303H508Q8B" package3d_urn="urn:adsk.eagle:package:23793141/1" value="SSCDRRV100MDSA3" x="43" y="50.333334375" smashed="yes" rot="R270"/>
+<element name="U$5" library="SCCDRRV100MDSA3" package="DIP1270W53P254L1303H508Q8B" package3d_urn="urn:adsk.eagle:package:23793141/1" value="SSCDRRV100MDSA3" x="58" y="40" smashed="yes" rot="R270"/>
 <element name="X1" library="con-JST XH" package="S4B-XH-A" value="S4B-XH-A" x="91" y="38" smashed="yes" rot="R270">
 <attribute name="NAME" x="78" y="35.202" size="1.016" layer="25" rot="R180" align="bottom-center"/>
@@
 <vertex x="100" y="80"/>
 </polygon>
-<wire x1="91" y1="34.25" x2="91" y2="47.25" width="0" layer="19" extent="1-1"/>
-<wire x1="82.4" y1="31.2" x2="91" y2="34.25" width="0" layer="19" extent="1-1"/>
-<wire x1="79.9" y1="26" x2="82.4" y2="31.2" width="0" layer="19" extent="1-1"/>
-<wire x1="82.4" y1="19.2" x2="79.9" y2="26" width="0" layer="19" extent="1-1"/>
-<wire x1="79.9" y1="14" x2="82.4" y2="19.2" width="0" layer="19" extent="1-1"/>
-<wire x1="72.125" y1="26.2178" x2="79.9" y2="26" width="0" layer="19" extent="1-1"/>
-<wire x1="71.475" y1="26.2178" x2="72.125" y2="26.2178" width="0" layer="19" extent="1-1"/>
-<wire x1="66.925" y1="26.2178" x2="71.475" y2="26.2178" width="0" layer="19" extent="1-1"/>
-<wire x1="71.475" y1="20.3822" x2="71.475" y2="26.2178" width="0" layer="19" extent="1-1"/>
-<wire x1="72.125" y1="20.3822" x2="71.475" y2="20.3822" width="0" layer="19" extent="1-1"/>
-<wire x1="70.175" y1="20.3822" x2="71.475" y2="20.3822" width="0" layer="19" extent="1-1"/>
-<wire x1="68.875" y1="20.3822" x2="70.175" y2="20.3822" width="0" layer="19" extent="1-1"/>
-<wire x1="67.575" y1="20.3822" x2="68.875" y2="20.3822" width="0" layer="19" extent="1-1"/>
-<wire x1="66.925" y1="20.3822" x2="67.575" y2="20.3822" width="0" layer="19" extent="1-1"/>
-<wire x1="61.81" y1="46.35" x2="66.925" y2="26.2178" width="0" layer="19" extent="1-1"/>
-<wire x1="46.81" y1="56.683334375" x2="61.81" y2="46.35" width="0" layer="19" extent="1-1"/>
-<wire x1="62.81" y1="67.016659375" x2="46.81" y2="56.683334375" width="0" layer="19" extent="1-1"/>
-<wire x1="46.81" y1="77.35" x2="62.81" y2="67.016659375" width="0" layer="19" extent="1-1"/>
-<wire x1="10.68" y1="26.08" x2="46.81" y2="56.683334375" width="0" layer="19" extent="1-1"/>
-<wire x1="10.68" y1="23.54" x2="10.68" y2="26.08" width="0" layer="19" extent="1-1"/>
-<wire x1="8.14" y1="26.08" x2="10.68" y2="26.08" width="0" layer="19" extent="1-1"/>
-<wire x1="5.6" y1="26.08" x2="8.14" y2="26.08" width="0" layer="19" extent="1-1"/>
-<wire x1="5.6" y1="28.62" x2="5.6" y2="26.08" width="0" layer="19" extent="1-1"/>
-<wire x1="10.68" y1="21" x2="10.68" y2="23.54" width="0" layer="19" extent="1-1"/>
-<wire x1="8.14" y1="23.54" x2="10.68" y2="23.54" width="0" layer="19" extent="1-1"/>
-<wire x1="5.6" y1="23.54" x2="5.6" y2="26.08" width="0" layer="19" extent="1-1"/>
-<wire x1="8.14" y1="21" x2="10.68" y2="21" width="0" layer="19" extent="1-1"/>
-<wire x1="5.6" y1="21" x2="5.6" y2="23.54" width="0" layer="19" extent="1-1"/>
 </signal>
 <signal name="5V">
