File: sensor card/sensor card.sch (EAGLE design)
At the start: 45 parts, among them J1 MJ-3536N, J2 MJ-3536N, U1 PCA9306, U2 MCP3008-I/SL, U3 MCP6064-E/SL, X1 S4B-XH-A, X2 S4B-XH-A

Commit message: small fixes
Parts:
- R16: MANUFACTURER-PART-NUMBER (none) -> RMCF0805FT16K5
- R17: MANUFACTURER-PART-NUMBER (none) -> RMCF0805FT100R
- R6: MANUFACTURER-PART-NUMBER (none) -> ERA-6ARB303V; SIMILAR-COMPONENTS (none) -> Vishay precision resistors or anything else that fits the s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
- R7: MANUFACTURER-PART-NUMBER (none) -> ERA-6ARB303V
- R8, R9: MANUFACTURER-PART-NUMBER (none) -> ERA-6ARB102V; SIMILAR-COMPONENTS (none) -> Vishay precision resistors or anything else that fits the s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
Changed lines of the file:
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@@
 <part name="U3" library="MCP6064-E_SL" deviceset="MCP6064-E/SL" device=""/>
 <part name="GND4" library="supply1" library_urn="urn:adsk.eagle:library:371" deviceset="GND" device=""/>
-<part name="R6" library="SparkFun-Passives" deviceset="RESISTOR" device="0805-RES" package3d_urn="urn:adsk.eagle:package:30824479/1" value="30k, 0.1%, 25ppm/C"/>
-<part name="R7" library="SparkFun-Passives" deviceset="RESISTOR" device="0805-RES" package3d_urn="urn:adsk.eagle:package:30824479/1" value="30k, 0.1%, 25ppm/C"/>
-<part name="R8" library="SparkFun-Passives" deviceset="RESISTOR" device="0805-RES" package3d_urn="urn:adsk.eagle:package:30824479/1" value="1k, 0.1%, 25ppm/C"/>
-<part name="R9" library="SparkFun-Passives" deviceset="RESISTOR" device="0805-RES" package3d_urn="urn:adsk.eagle:package:30824479/1" value="1k, 0.1%, 25ppm/C"/>
+<part name="R6" library="SparkFun-Passives" deviceset="RESISTOR" device="0805-RES" package3d_urn="urn:adsk.eagle:package:30824479/1" value="30k, 0.1%, 25ppm/C">
+<attribute name="MANUFACTURER-PART-NUMBER" value="ERA-6ARB303V"/>
+<attribute name="SIMILAR-COMPONENTS" value="Vishay precision resistors or anything else that fits the spec"/>
+</part>
+<part name="R7" library="SparkFun-Passives" deviceset="RESISTOR" device="0805-RES" package3d_urn="urn:adsk.eagle:package:30824479/1" value="30k, 0.1%, 25ppm/C">
+<attribute name="MANUFACTURER-PART-NUMBER" value="ERA-6ARB303V"/>
+</part>
+<part name="R8" library="SparkFun-Passives" deviceset="RESISTOR" device="0805-RES" package3d_urn="urn:adsk.eagle:package:30824479/1" value="1k, 0.1%, 25ppm/C">
+<attribute name="MANUFACTURER-PART-NUMBER" value="ERA-6ARB102V"/>
+<attribute name="SIMILAR-COMPONENTS" value="Vishay precision resistors or anything else that fits the spec"/>
+</part>
+<part name="R9" library="SparkFun-Passives" deviceset="RESISTOR" device="0805-RES" package3d_urn="urn:adsk.eagle:package:30824479/1" value="1k, 0.1%, 25ppm/C">
+<attribute name="MANUFACTURER-PART-NUMBER" value="ERA-6ARB102V"/>
+<attribute name="SIMILAR-COMPONENTS" value="Vishay precision resistors or anything else that fits the spec"/>
+</part>
 <part name="GND7" library="supply1" library_urn="urn:adsk.eagle:library:371" deviceset="GND" device=""/>
 <part name="GND8" library="supply1" library_urn="urn:adsk.eagle:library:371" deviceset="GND" device=""/>
@@
 <part name="P1" library="pinhead" library_urn="urn:adsk.eagle:library:325" deviceset="PINHD-1X1" device="" package3d_urn="urn:adsk.eagle:package:22485/2"/>
 <part name="P6" library="pinhead" library_urn="urn:adsk.eagle:library:325" deviceset="PINHD-1X1" device="" package3d_urn="urn:adsk.eagle:package:22485/2"/>
-<part name="R13" library="rcl" library_urn="urn:adsk.eagle:library:334" deviceset="R-TRIMM" device="3214W" package3d_urn="urn:adsk.eagle:package:23729/1">
+<part name="R13" library="rcl" deviceset="R-TRIMM" device="3214W" package3d_urn="urn:adsk.eagle:package:23729/1">
 <spice>
 <pinmapping spiceprefix="X">
@@
 <attribute name="PURCHASE" value="https://www.digikey.ca/en/products/detail/bourns-inc/3214W-1-502G/2535183"/>
 </part>
-<part name="R14" library="rcl" library_urn="urn:adsk.eagle:library:334" deviceset="R-TRIMM" device="3214W" package3d_urn="urn:adsk.eagle:package:23729/1">
+<part name="R14" library="rcl" deviceset="R-TRIMM" device="3214W" package3d_urn="urn:adsk.eagle:package:23729/1">
 <spice>
 <pinmapping spiceprefix="X">
@@
 <part name="GND15" library="supply1" library_urn="urn:adsk.eagle:library:371" deviceset="GND" device=""/>
 <part name="P7" library="pinhead" library_urn="urn:adsk.eagle:library:325" deviceset="PINHD-1X1" device="" package3d_urn="urn:adsk.eagle:package:22485/2"/>
-<part name="R16" library="SparkFun-Passives" deviceset="RESISTOR" device="0805-RES" package3d_urn="urn:adsk.eagle:package:30824479/1" value="16.5k, 1%"/>
-<part name="R17" library="SparkFun-Passives" deviceset="RESISTOR" device="0805-RES" package3d_urn="urn:adsk.eagle:package:30824479/1" value="100, 1%"/>
+<part name="R16" library="SparkFun-Passives" deviceset="RESISTOR" device="0805-RES" package3d_urn="urn:adsk.eagle:package:30824479/1" value="16.5k, 1%">
+<attribute name="MANUFACTURER-PART-NUMBER" value="RMCF0805FT16K5"/>
+</part>
+<part name="R17" library="SparkFun-Passives" deviceset="RESISTOR" device="0805-RES" package3d_urn="urn:adsk.eagle:package:30824479/1" value="100, 1%">
+<attribute name="MANUFACTURER-PART-NUMBER" value="RMCF0805FT100R"/>
+</part>
 <part name="GND9" library="supply1" library_urn="urn:adsk.eagle:library:371" deviceset="GND" device=""/>
 <part name="FRAME1" library="frames" library_urn="urn:adsk.eagle:library:229" deviceset="FRAME_B_L" device=""/>
