File: valves card/valves card.brd (EAGLE design)
At the start: 100 x 80 mm, 68 parts, among them J1 8-1393644-0, J2 TBP02R1-381-14BE, Q1 IRLZ44NSTRLPBF, Q11 IRLZ44NSTRLPBF, Q13 IRLZ44NSTRLPBF, Q15 IRLZ44NSTRLPBF, Q17 IRLZ44NSTRLPBF, Q19 IRLZ44NSTRLPBF, Q21 IRLZ44NSTRLPBF, Q23 IRLZ44NSTRLPBF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

Commit message: started bom creation
Routing:
- net SOL3: track 69.5 -> 70.5 mm
Changed lines of the file:
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@@
 <attribute name="DESCRIPTION" value="  Optoisolator Transistor Output 5000Vrms 1 Channel 4-DIP " x="53.5" y="47.8" size="1.778" layer="27" rot="R180" display="off"/>
 <attribute name="MF" value="Everlight" x="53.5" y="47.8" size="1.778" layer="27" rot="R180" display="off"/>
-<attribute name="MP" value="EL817(C)" x="53.5" y="47.8" size="1.778" layer="27" rot="R180" display="off"/>
+<attribute name="MP" value="OR-815" x="53.5" y="47.8" size="1.778" layer="27" rot="R180" display="off"/>
 <attribute name="NAME" x="23.604659375" y="9.19763125" size="1.271159375" layer="25" rot="R180"/>
 <attribute name="PACKAGE" value="DIP-4 Everlight" x="53.5" y="47.8" size="1.778" layer="27" rot="R180" display="off"/>
@@
 <wire x1="37" y1="42" x2="33" y2="46" width="0.4064" layer="16"/>
 <wire x1="37" y1="31" x2="37" y2="42" width="0.4064" layer="16"/>
-<via x="16.053021875" y="46.946978125" extent="1-16" drill="0.35"/>
+<via x="15.453021875" y="46.346978125" extent="1-16" drill="0.35"/>
 <wire x1="30.62013125" y1="46" x2="30.02553125" y2="46.5946" width="0.3048" layer="1"/>
-<wire x1="16.4054" y1="46.5946" x2="16.053021875" y2="46.946978125" width="0.3048" layer="1"/>
-<wire x1="30.02553125" y1="46.5946" x2="16.4054" y2="46.5946" width="0.3048" layer="1"/>
-<wire x1="16.053021875" y1="46.946978125" x2="16.053021875" y2="53.726978125" width="0.3048" layer="16"/>
-<wire x1="16.053021875" y1="53.726978125" x2="14.27" y2="55.51" width="0.3048" layer="16"/>
+<wire x1="15.70064375" y1="46.5946" x2="15.453021875" y2="46.346978125" width="0.3048" layer="1"/>
+<wire x1="30.02553125" y1="46.5946" x2="15.70064375" y2="46.5946" width="0.3048" layer="1"/>
+<wire x1="15.453021875" y1="46.346978125" x2="15.553021875" y2="46.446978125" width="0.3048" layer="16"/>
+<wire x1="15.553021875" y1="54.226978125" x2="15.553021875" y2="46.446978125" width="0.3048" layer="16"/>
+<wire x1="15.553021875" y1="54.226978125" x2="14.27" y2="55.51" width="0.3048" layer="16"/>
 <wire x1="33" y1="46" x2="32.0884" y2="46" width="0.3048" layer="16"/>
 <wire x1="32.0884" y1="46" x2="32" y2="45.9116" width="0.3048" layer="16"/>

Commit message: fixed library attributes for the din41612 connector, fixed git problems
Parts:
- J1: value 8-1393644-0 -> 09231486921; device 8-1393644-0:TE_8-1393644-0 -> din41612_48_pin_board:HARTING_09231486921
Changed lines of the file:
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@@
 </autorouter>
 <elements>
-<element name="J1" library="8-1393644-0" package="TE_8-1393644-0" value="8-1393644-0" x="5.6" y="21" smashed="yes" rot="R270">
+<element name="J1" library="din41612_48_pin_board" package="HARTING_09231486921" value="09231486921" x="5.6" y="21" smashed="yes" rot="R270">
 <attribute name="AVAILABILITY" value="In Stock" x="5.6" y="21" size="1.778" layer="27" rot="R270" display="off"/>
-<attribute name="COMMENT" value="8-1393644-0" x="5.6" y="21" size="1.778" layer="27" rot="R270" display="off"/>
+<attribute name="COMMENT" value="09231486921" x="5.6" y="21" size="1.778" layer="27" rot="R270" display="off"/>
 <attribute name="DESCRIPTION" value=" Conn DIN 41612 M 48 POS 2.54mm Solder RA Thru-Hole Tray " x="5.6" y="21" size="1.778" layer="27" rot="R270" display="off"/>
 <attribute name="EU_ROHS_COMPLIANCE" value="Compliant" x="5.6" y="21" size="1.778" layer="27" rot="R270" display="off"/>
-<attribute name="MF" value="TE Connectivity" x="5.6" y="21" size="1.778" layer="27" rot="R270" display="off"/>
-<attribute name="MP" value="8-1393644-0" x="5.6" y="21" size="1.778" layer="27" rot="R270" display="off"/>
+<attribute name="MF" value="HARTING" x="5.6" y="21" size="1.778" layer="27" rot="R270" display="off"/>
+<attribute name="MP" value="09231486921" x="5.6" y="21" size="1.778" layer="27" rot="R270" display="off"/>
 <attribute name="NAME" x="12.605" y="67.73" size="1.27" layer="25" rot="R270"/>
 <attribute name="PACKAGE" value="None" x="5.6" y="21" size="1.778" layer="27" rot="R270" display="off"/>
-<attribute name="PRICE" value="None" x="5.6" y="21" size="1.778" layer="27" rot="R270" display="off"/>
-<attribute name="PURCHASE-URL" value="https://pricing.snapeda.com/search/part/8-1393644-0/?ref=eda" x="5.6" y="21" size="1.778" layer="27" rot="R270" display="off"/>
+<attribute name="PRICE" value="6$" x="5.6" y="21" size="1.778" layer="27" rot="R270" display="off"/>
+<attribute name="PURCHASE-URL-DIGIKEY" value="https://www.digikey.ca/en/products/detail/harting/09231486921/3180439" x="5.6" y="21" size="1.778" layer="27" rot="R270" display="off"/>
 <attribute name="VALUE" x="-8.59" y="67.73" size="1.27" layer="27" rot="R270"/>
 </element>

Commit message: added cam data
Parts:
- Q1, Q11, Q13, Q15, Q17, Q19, Q21, Q23, Q3, Q5, Q7, Q9: device m_transistor:TO-252 -> BUK9214-30A,118:DPAK_TO252
- moved Q1 1.00 mm to (19.0, 21.0)
- moved Q11 1.00 mm to (37.0, 44.0)
- moved Q13 1.00 mm to (51.0, 44.0)
- moved Q15 1.00 mm to (66.0, 44.0)
- moved Q17 1.00 mm to (81.0, 44.0)
- moved Q19 1.00 mm to (49.0, 65.0)
- moved Q21 1.00 mm to (64.0, 65.0)
- moved Q23 1.00 mm to (79.0, 65.0)
- moved Q3 1.00 mm to (34.0, 21.0)
- moved Q5 1.00 mm to (49.0, 21.0)
- moved Q7 1.00 mm to (64.0, 21.0)
- moved Q9 1.00 mm to (79.0, 21.0)
Connections:
- removed net VCC: U$1.4@JP2
- net 3.3V: now also U$1.4@JP2
- net DRAIN1: now also Q1.2; no longer Q1.P$2
- net DRAIN10: now also Q19.2; no longer Q19.P$2
- net DRAIN11: now also Q21.2; no longer Q21.P$2
- net DRAIN12: now also Q23.2; no longer Q23.P$2
- net DRAIN2: now also Q3.2; no longer Q3.P$2
- net DRAIN3: now also Q5.2; no longer Q5.P$2
- net DRAIN4: now also Q7.2; no longer Q7.P$2
- net DRAIN5: now also Q9.2; no longer Q9.P$2
- net DRAIN6: now also Q11.2; no longer Q11.P$2
- net DRAIN7: now also Q13.2; no longer Q13.P$2
- net DRAIN8: now also Q15.2; no longer Q15.P$2
- net DRAIN9: now also Q17.2; no longer Q17.P$2
- net GND: now also Q1.3, Q11.3, Q13.3, Q15.3, Q17.3, Q19.3, Q21.3, Q23.3, Q3.3, Q5.3, Q7.3, Q9.3; no longer Q1.P$3, Q11.P$3, Q13.P$3, Q15.P$3, Q17.P$3, Q19.P$3, Q21.P$3, Q23.P$3, Q3.P$3, Q5.P$3, Q7.P$3, Q9.P$3
- net N$10: now also Q1.1; no longer Q1.P$1
- net N$15: now also Q3.1; no longer Q3.P$1
- net N$21: now also Q5.1; no longer Q5.P$1
- net N$27: now also Q7.1; no longer Q7.P$1
- net N$33: now also Q9.1; no longer Q9.P$1
- net N$39: now also Q11.1; no longer Q11.P$1
- net N$45: now also Q13.1; no longer Q13.P$1
- net N$51: now also Q15.1; no longer Q15.P$1
- net N$57: now also Q17.1; no longer Q17.P$1
- net N$63: now also Q19.1; no longer Q19.P$1
- net N$69: now also Q21.1; no longer Q21.P$1
- net N$75: now also Q23.1; no longer Q23.P$1
Routing:
- net 3.3V: track 0.00 -> 47.3 mm, vias 0 -> 1
- net GND: track 152.8 -> 150.1 mm
- net DRAIN6: track 71.0 -> 71.6 mm
- net DRAIN4: track 32.7 -> 32.1 mm
- net SOL9: track 76.1 -> 75.5 mm
- net N$69: track 6.88 -> 6.30 mm
- net N$63: track 6.88 -> 6.30 mm

Commit message: added cam data, and ordered pcb's based on that cam data, will clean up repo next
Parts:
- U2: value OR-815 -> EL817(D)-ND
Changed lines of the file:
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@@
 <attribute name="VALUE" x="-8.59" y="67.73" size="1.27" layer="27" rot="R270"/>
 </element>
-<element name="U2" library="EL817C" package="DIP762W25P254L650H453Q4B" value="OR-815" x="18.5" y="11.8" smashed="yes" rot="R180">
+<element name="U2" library="EL817C" package="DIP762W25P254L650H453Q4B" value="EL817(D)-ND" x="18.5" y="11.8" smashed="yes" rot="R180">
 <attribute name="AVAILABILITY" value="Bad" x="53.5" y="47.8" size="1.778" layer="27" rot="R180" display="off"/>
+<attribute name="BEST_I_COULD_FIND" value="EL817(D)-ND" x="18.5" y="11.8" size="1.778" layer="27" rot="R180" display="off"/>
 <attribute name="DESCRIPTION" value="  Optoisolator Transistor Output 5000Vrms 1 Channel 4-DIP " x="53.5" y="47.8" size="1.778" layer="27" rot="R180" display="off"/>
 <attribute name="MF" value="Everlight" x="53.5" y="47.8" size="1.778" layer="27" rot="R180" display="off"/>

Commit message: added libraries
Connections:
- net N$150 renamed 24V
Changed lines of the file:
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@@
 </layers>
 <board>
+<fusionsync huburn="a.cGVyc29uYWw6dWUyYTJjODE0" projecturn="a.cGVyc29uYWw6dWUyYWFmMDMwIzIwMjAwODE1MzIzNjg3MzAx" f3durn="urn:adsk.wipprod:dm.lineage:qNhJGBfgQ0mSe4L_LkHI8g" pcbguid="81a7e88e-a544-478a-828f-9ae69a135e87" lastpulledtime="" lastsyncedchangeguid="" latestrevisionid="0e11d027-5972-4da6-bd9e-e80dec3f924d" lastsyncedrevisionid="0e11d027-5972-4da6-bd9e-e80dec3f924d" lastboardhashguid="10dd5cbf-2d28-42bb-8bd6-ccc65134bc0e" lastpushedtime="2021-09-24T20:22:37Z" linktopcb3d="true"/>
 <plain>
 <wire x1="0" y1="0" x2="100" y2="0" width="0" layer="20"/>
@@
 <wire x1="72.8396" y1="62.52354375" x2="72.8396" y2="58.2396" width="1.016" layer="1"/>
 </signal>
-<signal name="N$150" class="1">
+<signal name="24V" class="1">
 <contactref element="J1" pad="5"/>
 <contactref element="J1" pad="6"/>
@@
 </note>
 <note version="8.3" severity="warning">
+Since Version 8.3, EAGLE supports Fusion synchronisation.
+This feature will not be available in this version and saving
+the document will break the link to the Fusion PCB feature.
+</note>
+<note version="8.3" severity="warning">
