File: backplane/backplane.sch (EAGLE design)
At the start: 10 parts, among them J1 09232486825, J10 TB009-508-05BE, J2 09232486825, J3 09232486825, J4 09232486825, J5 09232486825, J6 09232486825, J7 09232486825, J8 09232486825

Commit message: updated libraries to generate better bom's
Parts:
- JP2: IGNORE-IN-BOM (none) -> True
Changed lines of the file:
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@@
 <part name="GND4" library="supply1" library_urn="urn:adsk.eagle:library:371" deviceset="GND" device=""/>
 <part name="GND6" library="supply1" library_urn="urn:adsk.eagle:library:371" deviceset="GND" device=""/>
-<part name="JP2" library="pinhead" library_urn="urn:adsk.eagle:library:325" deviceset="PINHD-2X15" device="" package3d_urn="urn:adsk.eagle:package:22427/2"/>
+<part name="JP2" library="pinhead" library_urn="urn:adsk.eagle:library:325" deviceset="PINHD-2X15" device="" package3d_urn="urn:adsk.eagle:package:22427/2">
+<attribute name="IGNORE-IN-BOM" value="True"/>
+</part>
 <part name="J10" library="TB009-508-05BE" deviceset="TB009-508-05BE" device=""/>
 </parts>
@@
 <attribute name="NAME" x="-52.07" y="81.915" size="1.778" layer="95"/>
 <attribute name="VALUE" x="-52.07" y="38.1" size="1.778" layer="96"/>
+<attribute name="IGNORE-IN-BOM" x="-45.72" y="60.96" size="1.778" layer="96" display="off"/>
 </instance>
 <instance part="J10" gate="G$1" x="-48.26" y="96.52" smashed="yes" rot="R180">

Commit message: small fixes
Connections:
- net 3.3V: now also J10.1; no longer J10.5
- net 5V: now also J10.2; no longer J10.4
- net GND: now also J10.4, J10.5; no longer J10.1, J10.2
Other:
- moved on the sheet: J10
Changed lines of the file:
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@@
 <part name="GND2" library="supply1" library_urn="urn:adsk.eagle:library:371" deviceset="GND" device=""/>
 <part name="GND3" library="supply1" library_urn="urn:adsk.eagle:library:371" deviceset="GND" device=""/>
-<part name="GND4" library="supply1" library_urn="urn:adsk.eagle:library:371" deviceset="GND" device=""/>
 <part name="GND6" library="supply1" library_urn="urn:adsk.eagle:library:371" deviceset="GND" device=""/>
 <part name="JP2" library="pinhead" library_urn="urn:adsk.eagle:library:325" deviceset="PINHD-2X15" device="" package3d_urn="urn:adsk.eagle:package:22427/2">
@@
 </part>
 <part name="J10" library="TB009-508-05BE" deviceset="TB009-508-05BE" device=""/>
+<part name="GND5" library="supply1" library_urn="urn:adsk.eagle:library:371" deviceset="GND" device=""/>
 </parts>
 <sheets>
@@
 <attribute name="VALUE" x="-22.86" y="33.02" size="1.778" layer="96"/>
 </instance>
-<instance part="GND4" gate="1" x="-35.56" y="88.9" smashed="yes">
-<attribute name="VALUE" x="-38.1" y="86.36" size="1.778" layer="96"/>
-</instance>
 <instance part="GND6" gate="1" x="-66.04" y="76.2" smashed="yes">
 <attribute name="VALUE" x="-68.58" y="73.66" size="1.778" layer="96"/>
@@
 <attribute name="IGNORE-IN-BOM" x="-45.72" y="60.96" size="1.778" layer="96" display="off"/>
 </instance>
-<instance part="J10" gate="G$1" x="-48.26" y="96.52" smashed="yes" rot="R180">
-<attribute name="NAME" x="-42.68" y="88.9" size="1.778" layer="95" rot="R180"/>
-<attribute name="VALUE" x="-43.18" y="106.68" size="1.778" layer="96" rot="R180"/>
+<instance part="J10" gate="G$1" x="-48.26" y="96.52" smashed="yes">
+<attribute name="NAME" x="-53.84" y="104.14" size="1.778" layer="95"/>
+<attribute name="VALUE" x="-53.34" y="86.36" size="1.778" layer="96"/>
+</instance>
+<instance part="GND5" gate="1" x="-66.04" y="88.9" smashed="yes">
+<attribute name="VALUE" x="-68.58" y="86.36" size="1.778" layer="96"/>
 </instance>
 </instances>
@@
 </segment>
 <segment>
-<wire x1="-35.56" y1="93.98" x2="-35.56" y2="91.44" width="0.1524" layer="91"/>
-<pinref part="GND4" gate="1" pin="GND"/>
-<pinref part="J10" gate="G$1" pin="2"/>
-<pinref part="J10" gate="G$1" pin="1"/>
-<wire x1="-35.56" y1="91.44" x2="-38.1" y2="91.44" width="0.1524" layer="91"/>
-<junction x="-35.56" y="91.44"/>
-<wire x1="-38.1" y1="93.98" x2="-35.56" y2="93.98" width="0.1524" layer="91"/>
-</segment>
-<segment>
 <wire x1="-66.04" y1="78.74" x2="-48.26" y2="78.74" width="0.1524" layer="91"/>
 <pinref part="JP2" gate="A" pin="1"/>
 <pinref part="GND6" gate="1" pin="GND"/>
+</segment>
+<segment>
+<wire x1="-66.04" y1="93.98" x2="-66.04" y2="91.44" width="0.1524" layer="91"/>
+<pinref part="GND5" gate="1" pin="GND"/>
+<pinref part="J10" gate="G$1" pin="4"/>
+<wire x1="-58.42" y1="93.98" x2="-66.04" y2="93.98" width="0.1524" layer="91"/>
+<pinref part="J10" gate="G$1" pin="5"/>
+<wire x1="-66.04" y1="91.44" x2="-58.42" y2="91.44" width="0.1524" layer="91"/>
+<junction x="-66.04" y="91.44"/>
 </segment>
 </net>
@@
 </segment>
 <segment>
-<wire x1="-38.1" y1="96.52" x2="-27.94" y2="96.52" width="0.1524" layer="91"/>
-<label x="-38.1" y="96.52" size="1.778" layer="95"/>
+<wire x1="-68.58" y1="96.52" x2="-58.42" y2="96.52" width="0.1524" layer="91"/>
 <pinref part="J10" gate="G$1" pin="3"/>
+<label x="-68.58" y="96.52" size="1.778" layer="95"/>
 </segment>
 </net>
@@
 </segment>
 <segment>
-<wire x1="-27.94" y1="101.6" x2="-38.1" y2="101.6" width="0.1524" layer="91"/>
-<label x="-38.1" y="101.6" size="1.778" layer="95"/>
-<pinref part="J10" gate="G$1" pin="5"/>
-</segment>
-<segment>
 <pinref part="JP2" gate="A" pin="5"/>
 <wire x1="-48.26" y1="73.66" x2="-60.96" y2="73.66" width="0.1524" layer="91"/>
 <label x="-60.96" y="73.66" size="1.778" layer="95"/>
+</segment>
+<segment>
+<wire x1="-58.42" y1="101.6" x2="-68.58" y2="101.6" width="0.1524" layer="91"/>
+<pinref part="J10" gate="G$1" pin="1"/>
+<label x="-66.04" y="101.6" size="1.778" layer="95"/>
 </segment>
 </net>
@@
 </net>
 <net name="5V" class="0">
-<segment>
-<wire x1="-38.1" y1="99.06" x2="-27.94" y2="99.06" width="0.1524" layer="91"/>
-<label x="-38.1" y="99.06" size="1.778" layer="95"/>
-<pinref part="J10" gate="G$1" pin="4"/>
-</segment>
 <segment>
 <pinref part="J8" gate="G$1" pin="C7"/>
@@
 <label x="-60.96" y="76.2" size="1.778" layer="95"/>
 </segment>
-</net>
+<segment>
+<wire x1="-68.58" y1="99.06" x2="-58.42" y2="99.06" width="0.1524" layer="91"/>
+<pinref part="J10" gate="G$1" pin="2"/>
+<label x="-66.04" y="99.06" size="1.778" layer="95"/>
+</segment>
+</net>
