File: cards/sensor_card/board/sensor card.brd (EAGLE design)
At the start: 100 x 80 mm, 45 parts, among them J1 MJ-3536N, J2 MJ-3536N, U1 PCA9306, U2 MCP3008-I/SL, U3 MCP6064-E/SL, X1 S4B-XH-A, X2 S4B-XH-A

Commit message: fixed the emi cap footprint on the sensing card
Routing:
- net CH2: track 66.5 -> 74.3 mm
Other:
- board text added: "NOT DONE YET, NEEDS I2C CHANGES AND A BUG FIXED TO WORK (will be V1.2 then)"
Changed lines of the file:
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@@
 <drawing>
 <settings>
-<setting alwaysvectorfont="no"/>
+<setting alwaysvectorfont="yes"/>
 <setting verticaltext="up"/>
 </settings>
@@
 <text x="72" y="51" size="1.778" layer="25">25mV</text>
 <text x="72" y="36" size="1.778" layer="25">2V</text>
+<text x="-77" y="28" size="10" layer="25">NOT DONE YET, NEEDS I2C CHANGES AND A BUG FIXED TO WORK (will be V1.2 then)</text>
 </plain>
 <attributes>
@@
 <wire x1="61.02268125" y1="19.4202" x2="60.41788125" y2="20.025" width="0.3048" layer="1"/>
 <wire x1="66" y1="35" x2="60" y2="29" width="0.508" layer="1"/>
-<wire x1="60" y1="21" x2="59.1266" y2="20.1266" width="0.508" layer="1"/>
 <wire x1="59.1266" y1="20.1266" x2="59.09345" y2="20.1266" width="0.508" layer="1"/>
 <wire x1="59.09345" y1="20.1266" x2="58.99185" y2="20.025" width="0.508" layer="1"/>
 <wire x1="58.99185" y1="20.025" x2="58.145" y2="20.025" width="0.508" layer="1"/>
-<wire x1="60" y1="29" x2="60" y2="21" width="0.508" layer="1"/>
 <wire x1="86.785" y1="43.56" x2="86.2379" y2="43.56" width="0.508" layer="1"/>
 <wire x1="86.2379" y1="43.56" x2="85.2914" y2="42.6135" width="0.508" layer="1"/>
@@
 <wire x1="65" y1="20.33288125" x2="65" y2="21.91" width="0.3048" layer="1"/>
 <wire x1="65.2" y1="22.11" x2="66.16" y2="22.11" width="0.3048" layer="1"/>
+<wire x1="56.63" y1="29" x2="55.33" y2="27.7" width="0.508" layer="1"/>
+<wire x1="55.33" y1="27.7" x2="55.33" y2="26.4" width="0.508" layer="1"/>
+<wire x1="59.05" y1="25.06" x2="60.71" y2="23.4" width="0.508" layer="1"/>
+<wire x1="60.71" y1="23.4" x2="60.71" y2="21.71" width="0.508" layer="1"/>
+<wire x1="60" y1="29" x2="56.63" y2="29" width="0.508" layer="1"/>
+<wire x1="55.33" y1="26.4" x2="56.67" y2="25.06" width="0.508" layer="1"/>
+<wire x1="56.67" y1="25.06" x2="59.05" y2="25.06" width="0.508" layer="1"/>
+<wire x1="60.71" y1="21.71" x2="59.1266" y2="20.1266" width="0.508" layer="1"/>
 </signal>
 <signal name="CH7">

Commit message: fixed problems with control module 2.2, all boards are now ready to order
Routing:
- net GND: track 32.8 -> 40.0 mm, vias 17 -> 16
- net 5V: track 147.7 -> 146.3 mm
Other:
- board text added: "PolyVent Sensor Board V1.2 Public invention - Nathaniel Bechard Liscenced under: CERN OHL 2.0"
- board text removed: "NOT DONE YET, NEEDS I2C CHANGES AND A BUG FIXED TO WORK (will be V1.2 then)"
- board text removed: "PolyVent Sensor Board V1.1 Public invention - Nathaniel Bechard Liscenced under: CERN OHL 2.0"
Changed lines of the file:
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@@
 <text x="31.82" y="39.43" size="1.4" layer="25">P_EN3</text>
 <text x="31.82" y="43.18" size="1.4" layer="25">P_EN4</text>
-<text x="54.41" y="69.58" size="1.778" layer="25">PolyVent Sensor Board V1.1
+<text x="54.41" y="69.58" size="1.778" layer="25">PolyVent Sensor Board V1.2
 Public invention - Nathaniel Bechard
 Liscenced under: CERN OHL 2.0</text>
@@
 <text x="72" y="51" size="1.778" layer="25">25mV</text>
 <text x="72" y="36" size="1.778" layer="25">2V</text>
-<text x="-77" y="28" size="10" layer="25">NOT DONE YET, NEEDS I2C CHANGES AND A BUG FIXED TO WORK (will be V1.2 then)</text>
 </plain>
 <attributes>
@@
 <contactref element="U1" pad="P1"/>
 <contactref element="C1" pad="2"/>
-<wire x1="87.52" y1="63.06" x2="87.75" y2="62.88" width="0.3048" layer="1"/>
 <contactref element="U2" pad="14"/>
 <contactref element="U2" pad="9"/>
@@
 <wire x1="64.16" y1="44" x2="68" y2="44" width="0.508" layer="16"/>
 <via x="68" y="44" extent="1-16" drill="0.35"/>
-<wire x1="72.37" y1="9.43" x2="73.27" y2="8.53" width="0.508" layer="1"/>
-<wire x1="73.27" y1="8.53" x2="73.27" y2="8.24" width="0.508" layer="1"/>
-<via x="73.27" y="8.24" extent="1-16" drill="0.35"/>
+<wire x1="72.37" y1="9.43" x2="73.8" y2="8" width="0.508" layer="1"/>
+<wire x1="73.8" y1="8" x2="77" y2="8" width="0.508" layer="1"/>
+<wire x1="77" y1="8" x2="79" y2="6" width="0.508" layer="1"/>
+<wire x1="79" y1="6" x2="79" y2="5" width="0.508" layer="1"/>
 </signal>
 <signal name="5V">
@@
 <wire x1="83" y1="60" x2="84" y2="59" width="0.3048" layer="16"/>
 <wire x1="84" y1="59" x2="92" y2="59" width="0.3048" layer="16"/>
-<wire x1="98" y1="48.75" x2="97" y2="47.75" width="0.3048" layer="1"/>
 <via x="92" y="59" extent="1-16" drill="0.35"/>
 <wire x1="92" y1="59" x2="93.29" y2="57.71" width="0.3048" layer="16"/>
@@
 <wire x1="92.13" y1="61.42" x2="92.18" y2="59.18" width="0.3048" layer="1"/>
 <wire x1="92.18" y1="59.18" x2="92" y2="59" width="0.3048" layer="1"/>
-<wire x1="97.479" y1="51.4064" x2="98.1564" y2="50.729" width="0.508" layer="1"/>
-<wire x1="93.29" y1="54.57" x2="96.4536" y2="51.4064" width="0.508" layer="1"/>
-<wire x1="96.4536" y1="51.4064" x2="97.479" y2="51.4064" width="0.508" layer="1"/>
 <wire x1="98.1564" y1="48.9064" x2="97" y2="47.75" width="0.508" layer="1"/>
-<wire x1="98.1564" y1="50.729" x2="98.1564" y2="48.9064" width="0.508" layer="1"/>
 <wire x1="93.29" y1="54.57" x2="91.98" y2="55.88" width="0.508" layer="1"/>
 <wire x1="91.98" y1="55.88" x2="91.72" y2="55.88" width="0.508" layer="1"/>
@@
 <wire x1="66" y1="42" x2="60" y2="36" width="0.508" layer="1"/>
 <wire x1="66" y1="46" x2="66" y2="42" width="0.508" layer="1"/>
+<wire x1="97.389" y1="51.4964" x2="98.1564" y2="50.729" width="0.508" layer="1"/>
+<wire x1="93.29" y1="54.57" x2="96.3636" y2="51.4964" width="0.508" layer="1"/>
+<wire x1="96.3636" y1="51.4964" x2="97.389" y2="51.4964" width="0.508" layer="1"/>
+<wire x1="98.1564" y1="50.729" x2="98.1564" y2="48.9064" width="0.508" layer="1"/>
 </signal>
 <signal name="3.3V">
@@
 <wire x1="8.526175" y1="42.3788" x2="7.701425" y2="42.3788" width="0.3048" layer="16"/>
 <wire x1="7.701425" y1="42.3788" x2="7" y2="41.677375" width="0.3048" layer="16"/>
-<wire x1="30.27" y1="70.27" x2="30" y2="70" width="0.3048" layer="1"/>
 <wire x1="30" y1="70" x2="27" y2="67" width="0.3048" layer="1"/>
 <wire x1="27" y1="67" x2="27" y2="51.7493125" width="0.3048" layer="1"/>
@@
 <wire x1="50.173340625" y1="62" x2="55.19" y2="67.016659375" width="0.3048" layer="16"/>
 <wire x1="43.38" y1="62" x2="50.173340625" y2="62" width="0.3048" layer="16"/>
-<wire x1="55.19" y1="67.016659375" x2="49.206659375" y2="73" width="0.3048" layer="16"/>
-<wire x1="34.08" y1="73" x2="33.19" y2="73.89" width="0.3048" layer="16"/>
-<wire x1="34.08" y1="73" x2="49.206659375" y2="73" width="0.3048" layer="16"/>
+<wire x1="55.19" y1="67.016659375" x2="50.206659375" y2="72" width="0.3048" layer="16"/>
+<wire x1="35.08" y1="72" x2="33.19" y2="73.89" width="0.3048" layer="16"/>
+<wire x1="35.08" y1="72" x2="50.206659375" y2="72" width="0.3048" layer="16"/>
 <wire x1="29.317" y1="47.2829125" x2="29.7170875" y2="47.683" width="0.3048" layer="16"/>
 <wire x1="26.6068" y1="43.6068" x2="29.317" y2="46.317" width="0.3048" layer="16"/>
